File: pcb/output/apriltag_cam.kicad_pcb (KiCad board)
At the start: 4 copper layers, 48 x 48 mm, 152 parts, among them J1 USB-C, J2 JTAG, SW1 BOOTSEL, U1 LFE5U-45F-8BG381C, U10 OV9281, U11 USBLC6-2SC6, U2 RP2350A, U3 W25Q128JVSIQ, U4 TLV62569, U5 TLV62569, U6 TLV75525, U7 TLV75518, U8 TLV75528, U9 TLV75512, Y1 12MHz, Y2 24MHz 1.8V

Commit message: Sourcing: U1 to LFE5U-25F-8BG381I (speed 8, in stock), BOM, production docs, 25F/85F timing sweep
Co-Authored-By: Claude Sonnet 5.5 <noreply@anthropic.com>
Parts:
- U1: value LFE5U-45F-8BG381C -> LFE5U-25F-8BG381I
Changed lines of the file:
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@@
 			)
 		)
-		(property "Value" "LFE5U-45F-8BG381C"
+		(property "Value" "LFE5U-25F-8BG381I"
 			(at 0 -9.5 90)
 			(layer "B.Fab")
