File: pcb/output/apriltag_cam.kicad_pcb (KiCad board)
At the start: 4 copper layers, 48 x 48 mm, 152 parts, among them J1 USB-C, J2 JTAG, SW1 BOOTSEL, U1 LFE5U-25F-8BG381I, U10 OV9281, U11 USBLC6-2SC6, U2 RP2350A, U3 W25Q128JVSIQ, U4 TLV62569, U5 TLV62569, U6 TLV75525, U7 TLV75518, U8 TLV75528, U9 TLV75512, Y1 12MHz, Y2 24MHz 1.8V

Commit message: PCB: connect floating power pads, in-stock LDOs, flash MPN, 1.9 mm screw holes, ERC tests
DRC 69+10 unconnected -> 67+0. Co-Authored-By: Claude Sonnet 5.5 <noreply@anthropic.com>
Parts:
- U3: value W25Q128JVSIQ -> W25Q128JVPIQ
- U6: value TLV75525 -> ME6211C25
- U8: value TLV75528 -> ME6211C28
- Y1: value 12MHz -> 12MHz 10pF
Routing:
- net +3V3: track 57.4 -> 108.6 mm, vias 70 -> 73
- net QSPI_SD0: track 17.5 -> 20.4 mm
- net GND: track 175.4 -> 178.0 mm
